Commit message: Added realsense URDF. Isolated align_depth as the source of realsense issues.

File: urdf/f1tenth.urdf.xacro (robot description, xacro)
@@ -4,7 +4,7 @@
   <xacro:arg name="use_nominal_extrinsics" default="False" />
   <xacro:include filename="$(find realsense2_description)/urdf/_d435i.urdf.xacro"/>
-<!--  <link name="base_link" />-->
-  <xacro:sensor_d435i parent="base_link" use_nominal_extrinsics="$(arg use_nominal_extrinsics)" add_plug="False" use_mesh="True">
-<!--    <origin xyz="0.24115 0 0.0961" rpy="0 0 0"/>-->
+  <link name="base_link" />
+  <xacro:sensor_d435i parent="base_link" use_nominal_extrinsics="$(arg use_nominal_extrinsics)">
+    <origin xyz="0.24115 0 0.0961" rpy="0 0 0"/>
   </xacro:sensor_d435i>
 </robot>

Commit message: Made imu_corrector output frame dynamic. Updated sensor extrinsic transformations to latest values.

File: urdf/f1tenth.urdf.xacro (robot description, xacro)
@@ -4,7 +4,7 @@
   <xacro:arg name="use_nominal_extrinsics" default="False" />
   <xacro:include filename="$(find realsense2_description)/urdf/_d435i.urdf.xacro"/>
-  <link name="base_link" />
-  <xacro:sensor_d435i parent="base_link" use_nominal_extrinsics="$(arg use_nominal_extrinsics)">
-    <origin xyz="0.24115 0 0.0961" rpy="0 0 0"/>
+  <link name="sensor_kit_link" />
+  <xacro:sensor_d435i parent="sensor_kit_link" use_nominal_extrinsics="$(arg use_nominal_extrinsics)">
+    <origin xyz="0.1775164 0 0.0639086" rpy="0 0 0"/>
   </xacro:sensor_d435i>
 </robot>

Commit message: Updated imu_filter.launch.py and imu_corrector with dynamic names for the node and output topic so multiple IMUs can run the bias removal at once. Changed the default output frame of the filtered IMU data to a common origin, i.e. the sensor kit so the orientation and movements correspond to the cars movement/orientation. Also reduced the realsense framerate.

File: urdf/f1tenth.urdf.xacro (robot description, xacro)
@@ -6,5 +6,5 @@
   <link name="sensor_kit_link" />
   <xacro:sensor_d435i parent="sensor_kit_link" use_nominal_extrinsics="$(arg use_nominal_extrinsics)">
-    <origin xyz="0.1775164 0 0.0639086" rpy="0 0 0"/>
+    <origin xyz="0.1775164 0 0.0639086" rpy="0 0 0"/> <!-- set pitch=3.14159265 for correct IMU rotation -->
   </xacro:sensor_d435i>
 </robot>

Commit message: Reset default gyro offset for correction. Modified laser box filter range to remove the robot. Temporarily enabled AMCL tf broadcast while disabling EKF map. Updated nav2 costmap parameters [needs testing]. Enabled launching ICP odometry. Updated VESC and realsense IMU covariance values. Added more tfs to static transform tree.

File: urdf/f1tenth.urdf.xacro (robot description, xacro)
@@ -6,5 +6,5 @@
   <link name="sensor_kit_link" />
   <xacro:sensor_d435i parent="sensor_kit_link" use_nominal_extrinsics="$(arg use_nominal_extrinsics)">
-    <origin xyz="0.1775164 0 0.0639086" rpy="0 0 0"/> <!-- set pitch=3.14159265 for correct IMU rotation -->
+    <origin xyz="0.1775164 0 0.0639086" rpy="0 0 0"/>
   </xacro:sensor_d435i>
 </robot>
